Commit message: added camera files

File: src/ros_components_description/urdf/stereolabs_zed.urdf.xacro (robot description, xacro)
@@ -87,5 +87,6 @@
     <link name="${device_namespace}_center">
       <visual>
-        <origin xyz="${screw_offset_x} 0 ${screw_offset_z}" rpy="0 0 0" />
+        <!-- 0.02 in x is caused because the visual model is in the frame -->
+        <origin xyz="${screw_offset_x-0.02} 0 ${screw_offset_z}" rpy="0 0 0" />
         <geometry>
           <mesh filename="package://ros_components_description/meshes/${model}.stl" />
@@ -95,14 +96,15 @@
         </material>
       </visual>
-      <collision>
+      <!-- <collision>
         <geometry>
           <mesh filename="package://ros_components_description/meshes/${model}.stl" />
         </geometry>
-      </collision>
+      </collision>-->
     </link>
     <joint name="${device_namespace}_camera_center_joint" type="fixed">
       <parent link="${device_namespace}_link" />
       <child link="${device_namespace}_center" />
-      <origin xyz="0 0 ${height/2}" rpy="0 ${bottom_slope} 0" />
+      <!-- 0.02 in x is caused because the visual model is in the frame -->
+      <origin xyz="0.02 0 ${height/2}" rpy="0 ${bottom_slope} 0" />
     </joint>
     <!-- Artificially Created Camera Center -->
@@ -111,5 +113,6 @@
       <parent link="${device_namespace}_center" />
       <child link="${device_namespace}_center_optical_frame" />
-      <origin xyz="0.01 0 0" rpy="0 0 0" />
+     <origin xyz="0.0 0.0 0.0" rpy="${-pi/2.0} 0 ${-pi/2.0}" />
+       <!--     <origin xyz="0.0 0.0 0.0" rpy="0 0 0" />-->
     </joint>
     <!-- Left Camera -->
@@ -163,16 +166,16 @@
     camera
       should be more accurate different frames and fovs can be set -->
-    <gazebo reference="${device_namespace}_center_optical_frame">
+    <gazebo reference="${device_namespace}_center">
       <sensor type="camera" name="${ns}${device_namespace}_stereolabs_zed_color">
         <always_on>true</always_on>
-        <update_rate>30.0</update_rate>
+        <update_rate>15.0</update_rate>
         <topic>${ns}${device_namespace}/zed_node/rgb/image_rect_color</topic>
         <visualize>false</visualize>
-        <ignition_frame_id>${device_namespace}_center_optical_frame</ignition_frame_id>
+        <ignition_frame_id>${ns}${device_namespace}_center_optical_frame</ignition_frame_id>
         <camera>
           <horizontal_fov>${110.0/180.0*pi}</horizontal_fov>
           <image>
-            <width>1920</width>
-            <height>1080</height>
+            <width>960</width>
+            <height>640</height>
             <format>R8G8B8</format>
           </image>
@@ -183,4 +186,6 @@
         </camera>
       </sensor>
+  </gazebo>
+  <gazebo reference="${device_namespace}_center">
       <sensor type="depth_camera" name="${ns}${device_namespace}_stereolabs_zed_depth">
         <always_on>true</always_on>
@@ -188,10 +193,13 @@
         <topic>${ns}${device_namespace}/zed_node/depth</topic>
         <visualize>false</visualize>
-        <ignition_frame_id>${device_namespace}_center_optical_frame</ignition_frame_id>
+        <ignition_frame_id>${ns}${device_namespace}_center_optical_frame</ignition_frame_id>
         <camera>
           <horizontal_fov>${110.0/180.0*pi}</horizontal_fov>
           <image>
-            <width>1920</width>
-            <height>1080</height>
+           <!--  <width>1920</width>
+            <height>1080</height>-->
+            <!-- Better pointclound performance -->
+            <width>160</width>
+            <height>100</height>
             <format>R_FLOAT32</format>
           </image>
